Commit message: corrected caster pose & package names

File: urdf/base.urdf.xacro (robot description, xacro)
@@ -4,16 +4,16 @@
        xmlns:interface="http://playerstage.sourceforge.net/gazebo/xmlschema/#interface"
        xmlns:xacro="http://www.ros.org/wiki/xacro">
-  <xacro:include filename="$(find new_wheelchair)/urdf/wheelchair.gazebo.xacro" />
-  <xacro:include filename="$(find new_wheelchair)/urdf/wheelchair.transmission.xacro" />
-  <xacro:include filename="$(find new_wheelchair)/urdf/wheelchair.constants.xacro" />
-  <xacro:include filename="$(find new_wheelchair)/urdf/wheelchair.kinect.xacro" />
-  <xacro:include filename="$(find new_wheelchair)/urdf/wheelchair.hokuyo.xacro" />
+  <xacro:include filename="$(find nuric_wheelchair_model_02)/urdf/wheelchair.gazebo.xacro" />
+  <xacro:include filename="$(find nuric_wheelchair_model_02)/urdf/wheelchair.transmission.xacro" />
+  <xacro:include filename="$(find nuric_wheelchair_model_02)/urdf/wheelchair.constants.xacro" />
+  <xacro:include filename="$(find nuric_wheelchair_model_02)/urdf/wheelchair.kinect.xacro" />
+  <xacro:include filename="$(find nuric_wheelchair_model_02)/urdf/wheelchair.hokuyo.xacro" />
   <property name="PI" value="3.1415926535897931" />
   <property name="front_wheel_radius" value="0.17" />
-  <property name="front_wheel_base_y" value="0.3" />
+  <property name="front_wheel_base_y" value="0.27" />
   <property name="caster_wheel_radius" value="0.1" />
   <property name="caster_wheel_hub_y" value="0.0" />
   <property name="caster_wheel_hub_x" value="-0.06" />
-  <property name="caster_hub_base_x" value="-0.465" />
+  <property name="caster_hub_base_x" value="-0.58" />
   <property name="caster_hub_base_y" value="0.19" />
   <property name="caster_hub_base_z" value="-0.07" />
@@ -39,5 +39,5 @@
         <geometry>
           <!-- <cylinder length="0.07" radius="${front_wheel_radius}" /> -->
-          <mesh filename="package://new_wheelchair/meshes/front_wheel.dae" />
+          <mesh filename="package://nuric_wheelchair_model_02/meshes/front_wheel.dae" />
         </geometry>
       </visual>
@@ -46,5 +46,5 @@
         <geometry>
           <cylinder length="0.07" radius="${front_wheel_radius}" />
-          <!-- <mesh filename="package://new_wheelchair/meshes/front_wheel.dae" /> -->
+          <!-- <mesh filename="package://nuric_wheelchair_model_02/meshes/front_wheel.dae" /> -->
         </geometry>
       </collision>
@@ -69,5 +69,5 @@
         <geometry>
           <!-- <cylinder length="0.038" radius="${caster_wheel_radius}" /> -->
-          <mesh filename="package://new_wheelchair/meshes/caster_wheel.dae" />
+          <mesh filename="package://nuric_wheelchair_model_02/meshes/caster_wheel.dae" />
         </geometry>
       </visual>
@@ -76,5 +76,5 @@
         <geometry>
           <cylinder length="0.038" radius="${caster_wheel_radius}" />
-          <!-- <mesh filename="package://new_wheelchair/meshes/caster_wheel.dae" /> -->
+          <!-- <mesh filename="package://nuric_wheelchair_model_02/meshes/caster_wheel.dae" /> -->
          </geometry>
       </collision>
@@ -96,11 +96,11 @@
       <visual>
         <geometry>
-          <mesh filename="package://new_wheelchair/meshes/caster_hub_${suffix}.dae" />
-        </geometry>
-      </visual>
-      <collision>
-        <origin xyz="0 0 0" rpy="0 0 0" />
-        <geometry>
-          <mesh filename="package://new_wheelchair/meshes/caster_hub_${suffix}.dae" />
+          <mesh filename="package://nuric_wheelchair_model_02/meshes/caster_hub_${suffix}.dae" />
+        </geometry>
+      </visual>
+      <collision>
+        <origin xyz="0 0 0" rpy="0 0 0" />
+        <geometry>
+          <mesh filename="package://nuric_wheelchair_model_02/meshes/caster_hub_${suffix}.dae" />
         </geometry>
       </collision>
@@ -135,11 +135,11 @@
       <visual>
         <geometry>
-          <mesh filename="package://new_wheelchair/meshes/wheelchair_base_seat.dae" />
-        </geometry>
-      </visual>
-      <collision>
-        <origin xyz="0 0 0" rpy="0 0 0" />
-        <geometry>
-          <mesh filename="package://new_wheelchair/meshes/wheelchair_base_seat.dae" />
+          <mesh filename="package://nuric_wheelchair_model_02/meshes/wheelchair_base_seat.dae" />
+        </geometry>
+      </visual>
+      <collision>
+        <origin xyz="0 0 0" rpy="0 0 0" />
+        <geometry>
+          <mesh filename="package://nuric_wheelchair_model_02/meshes/wheelchair_base_seat.dae" />
         </geometry>
       </collision>
@@ -171,5 +171,5 @@
       <visual>
         <geometry>
-          <mesh filename="package://new_wheelchair/meshes/wheel.dae" />
+          <mesh filename="package://nuric_wheelchair_model_02/meshes/wheel.dae" />
         </geometry>
       </visual>

File: urdf/wheelchair.hokuyo.xacro (robot description, xacro)
@@ -23,5 +23,5 @@
      <origin xyz="0 0 0" rpy="0 0 0"/>
      <geometry>
-       <mesh filename="package://new_wheelchair/meshes/hokuyo.dae"/>
+       <mesh filename="package://nuric_wheelchair_model_02/meshes/hokuyo.dae"/>
      </geometry>
    </visual> -->

File: urdf/wheelchair.kinect.xacro (robot description, xacro)
@@ -65,5 +65,5 @@
       <origin xyz="0 0 0" rpy="0 0 0" />
       <geometry>
-        <mesh filename="package://new_wheelchair/meshes/kinect.dae"/>
+        <mesh filename="package://nuric_wheelchair_model_02/meshes/kinect.dae"/>
       </geometry>
     </visual> -->

File: urdf/wheelchair.urdf.xacro (robot description, xacro)
@@ -5,5 +5,5 @@
        xmlns:xacro="http://www.ros.org/wiki/xacro"
        name="wheelchair" >
-  <xacro:include filename="$(find new_wheelchair)/urdf/base.urdf.xacro" />
+  <xacro:include filename="$(find nuric_wheelchair_model_02)/urdf/base.urdf.xacro" />
   <xacro:wheelchair_base />
 </robot>
