Commit message: updated urdf w/ gazebo_ros_control to publish joint states

File: urdf/wheelchair.gazebo.xacro (robot description, xacro)
@@ -4,4 +4,12 @@
        xmlns:interface="http://playerstage.sourceforge.net/gazebo/xmlschema/#interface"
        xmlns:xacro="http://www.ros.org/wiki/xacro">
+  <gazebo>
+    <plugin name="gazebo_ros_control" filename="libgazebo_ros_control.so" />
+      <plugin filename="libgazebo_ros_joint_state_publisher.so" name="joint_state_publisher">
+        <jointName>base_left_caster_hub_joint, base_right_caster_hub_joint, base_left_front_wheel_joint, base_right_front_wheel_joint, left_caster_hub_left_caster_wheel_joint, right_caster_hub_right_caster_wheel_joint</jointName>
+        <updateRate>150.0</updateRate>
+        <alwaysOn>true</alwaysOn>
+      </plugin>
+  </gazebo>
   <xacro:macro name="front_wheel_gazebo" params="suffix" >
     <gazebo reference="${suffix}_front_wheel_link" >

File: urdf/wheelchair.transmission.xacro (robot description, xacro)
@@ -6,8 +6,12 @@
   <!--  Front wheel transmission   -->
   <xacro:macro name="front_wheel_transmission" params="suffix parent reflect">
-    <transmission type="pr2_mechanism_model/SimpleTransmission" name="${suffix}_front_wheel_trans">
-      <actuator name="${suffix}_front_wheel_motor" />
-      <joint name="${parent}_${suffix}_front_wheel_joint" />
-      <mechanicalReduction>${reflect*1.0}</mechanicalReduction>
+    <transmission name="${suffix}_front_wheel_trans">
+      <type>transmission_interface/SimpleTransmission</type>
+      <joint name="${parent}_${suffix}_front_wheel_joint" >
+        <hardwareInterface>EffortJointInterface</hardwareInterface>
+      </joint>
+      <actuator name="${suffix}_front_wheel_motor" >
+        <mechanicalReduction>${reflect*1.0}</mechanicalReduction>
+      </actuator>
     </transmission>
   </xacro:macro>

File: urdf/wheelchair.urdf.xacro (robot description, xacro)
@@ -1,8 +1,8 @@
 <?xml version="1.0"?>
-<robot xmlns:sensor="http://playerstage.sourceforge.net/gazebo/xmlschema/#sensor"
+<robot name="nuric_wheelchair_02"
+       xmlns:sensor="http://playerstage.sourceforge.net/gazebo/xmlschema/#sensor"
        xmlns:controller="http://playerstage.sourceforge.net/gazebo/xmlschema/#controller"
        xmlns:interface="http://playerstage.sourceforge.net/gazebo/xmlschema/#interface"
-       xmlns:xacro="http://www.ros.org/wiki/xacro"
-       name="wheelchair" >
+       xmlns:xacro="http://www.ros.org/wiki/xacro" >
   <xacro:include filename="$(find nuric_wheelchair_model_02)/urdf/base.urdf.xacro" />
   <xacro:wheelchair_base />
